Commit message: changes too much

File: hand_model/urdf/hand_model.urdf (robot description, URDF)
Before this commit: robot hand_model, 17 links, 16 joints
Joints:
- joint index_joint_1: limit lower=-2 upper=2 effort=15 velocity=137 -> lower=-1 upper=2 effort=15 velocity=137
- joint index_joint_2: limit lower=-2 upper=2 effort=15 velocity=137 -> lower=-1 upper=2 effort=15 velocity=137
- joint index_joint_3: limit lower=-2 upper=2 effort=15 velocity=137 -> lower=-1 upper=2 effort=15 velocity=137
- joint little_joint_1: limit lower=-2 upper=2 effort=15 velocity=137 -> lower=-1 upper=2 effort=15 velocity=137
- joint little_joint_2: limit lower=-2 upper=2 effort=15 velocity=137 -> lower=-1 upper=2 effort=15 velocity=137
- joint little_joint_3: limit lower=-2 upper=2 effort=15 velocity=137 -> lower=-1 upper=2 effort=15 velocity=137
- joint middle_joint_1: limit lower=-2 upper=2 effort=15 velocity=137 -> lower=-1 upper=2 effort=15 velocity=137
- joint middle_joint_2: limit lower=-2 upper=2 effort=15 velocity=137 -> lower=-1 upper=2 effort=15 velocity=137
- joint middle_joint_3: limit lower=-2 upper=2 effort=15 velocity=137 -> lower=-1 upper=2 effort=15 velocity=137
- joint ring_joint_1: limit lower=-2 upper=2 effort=15 velocity=137 -> lower=-1 upper=2 effort=15 velocity=137
- joint ring_joint_2: limit lower=-2 upper=2 effort=15 velocity=137 -> lower=-1 upper=2 effort=15 velocity=137
- joint ring_joint_3: limit lower=-2 upper=2 effort=15 velocity=137 -> lower=-1 upper=2 effort=15 velocity=137
- joint thumb_joint_1: limit lower=-2 upper=2 effort=15 velocity=137 -> lower=-1 upper=2 effort=15 velocity=137
- joint thumb_joint_2: limit lower=-2 upper=2 effort=15 velocity=137 -> lower=-1 upper=2 effort=15 velocity=137
- joint thumb_joint_3: limit lower=-2 upper=2 effort=15 velocity=137 -> lower=-1 upper=2 effort=15 velocity=137

File: universal_robot/ur_e_description/urdf/ur.camera.xacro (robot description, xacro)
@@ -4,11 +4,12 @@
       <color rgba="0.8 0.0 0.0 1.0"/>
     </material>
-    <xacro:property name="cameraSize" value="0.05" /> <!-- Size of square 'camera' box -->
+    <xacro:property name="cameraSize" value="0.02" /> <!-- Size of square 'camera' box -->
     <xacro:property name="cameraMass" value="0.1" /> <!-- Mass of square 'camera' box -->
-    <joint name="camera_joint" type="fixed">
-        <axis xyz="0 0 0" />
-        <origin xyz="0 0 1" rpy="0 0 0"/>
-        <parent link="upper_arm_link"/>
+    <joint name="camera_joint" type="revolute">
+        <axis xyz="0 1 0" />
+        <origin xyz="-0.3 0 0" rpy="0 0 ${-pi/2}"/>
+        <parent link="forearm_link"/>
         <child link="camera_link"/>
+        <limit lower="-2" upper="2" effort="330.0" velocity="3.14"/>
       </joint>
       <!-- Camera -->

File: universal_robot/ur_e_description/urdf/ur.gazebo.xacro (robot description, xacro)
@@ -20,4 +20,7 @@
       <selfCollide>true</selfCollide>
     </gazebo>
+    <gazebo reference="${prefix}camera_link">
+      <selfCollide>true</selfCollide>
+    </gazebo>
     <gazebo reference="${prefix}ee_link">
       <selfCollide>true</selfCollide>

File: universal_robot/ur_e_description/urdf/ur.transmission.xacro (robot description, xacro)
@@ -56,4 +56,13 @@
       </actuator>
     </transmission>
+    <transmission name="${prefix}camera_link_trans">
+      <type>transmission_interface/SimpleTransmission</type>
+      <joint name="${prefix}camera_joint">
+        <hardwareInterface>hardware_interface/EffortJointInterface</hardwareInterface>
+      </joint>
+      <actuator name="${prefix}camera_3_motor">
+        <mechanicalReduction>1</mechanicalReduction>
+      </actuator>
+    </transmission>
   </xacro:macro>
 </robot>

File: universal_robot/ur_e_description/urdf/ur10e.urdf.xacro (robot description, xacro)
@@ -25,4 +25,5 @@
     wrist_2_lower_limit:=${-pi}    wrist_2_upper_limit:=${pi}
     wrist_3_lower_limit:=${-pi}    wrist_3_upper_limit:=${pi}
+    camera_lower_limit:=${-pi}    camera_upper_limit:=${-pi}
     transmission_hw_interface:=hardware_interface/PositionJointInterface
     safety_limits:=false safety_pos_margin:=0.15

File: universal_robot/ur_e_description/urdf/ur10e_joint_limited_robot.urdf.xacro (robot description, xacro)
@@ -14,4 +14,5 @@
 		 wrist_2_lower_limit="${-pi}" wrist_2_upper_limit="${pi}"
 		 wrist_3_lower_limit="${-pi}" wrist_3_upper_limit="${pi}"
+     camera_lower_limit="${-pi}" camera_upper_limit="${pi}"
 />
   <link name="world" />
