Commit message: exo and hand are shown in Rviz and gazebo together

File: universal_robot/ur_e_description/urdf/ur.camera.xacro (robot description, xacro)
@@ -4,14 +4,25 @@
       <color rgba="0.8 0.0 0.0 1.0"/>
     </material>
-    <xacro:property name="cameraSize" value="0.02" /> <!-- Size of square 'camera' box -->
+    <xacro:property name="cameraSize" value="0.07" /> <!-- Size of square 'camera' box -->
     <xacro:property name="cameraMass" value="0.1" /> <!-- Mass of square 'camera' box -->
-    <joint name="camera_joint" type="revolute">
-        <axis xyz="0 1 0" />
-        <origin xyz="-0.3 0 0" rpy="0 0 ${-pi/2}"/>
-        <parent link="forearm_link"/>
+    <joint name="prismatic_joint_Z" type="prismatic">
+        <axis xyz="0 0 1" limit="-3.14 3.14" />
+        <origin xyz="0 0 1" rpy="0 0 0"/>
+        <parent link="base_link"/>
+        <child link="dummy_link1"/>
+        <limit effort="330.0" velocity="3.14"/>
+      </joint>
+      <link name="dummy_link1"/>
+      <joint name="base_link_to dummy_link1" type="fixed">
+        <parent link="base_link" />
+        <child link="dummy_link1" />
+      </joint>
+      <joint name="revolute_joint_z" type="revolute">
+        <axis xyz="0 0 1" limit="-3.14 3.14" />
+        <origin xyz="0 0 1" rpy="0 0 0"/>
+        <parent link="dummy_link1"/>
         <child link="camera_link"/>
-        <limit lower="-2" upper="2" effort="330.0" velocity="3.14"/>
+        <limit effort="330.0" velocity="3.14"/>
       </joint>
-      <!-- Camera -->
       <link name="camera_link">
         <collision>
@@ -35,3 +46,47 @@
         </inertial>
       </link>
+      <!-- <link name="dummy_link1"/>
+      <link name="dummy_link2"/>
+      <joint name="base_link_to dummy_link1" type="fixed">
+        <parent link="base_link" />
+        <child link="dummy_link1" />
+      </joint> -->
+      <!-- <joint name="base_link_to dummy_link2" type="fixed">
+        <parent link="world" />
+        <child link="dummy_link2" />
+      </joint>   -->
+      <!-- <joint name="prismatic_joint_Z" type="prismatic">
+        <parent link="base_link"/>
+        <child link="dummy_link1"/>
+        <origin xyz="0 0 1" rpy="0 0 0"/>
+        <axis xyz="0 0 1"/>
+        <limit lower="-2" upper="2" effort="50" velocity="3.49" />
+      </joint>
+      <joint name="revolute_joint_z" type="revolute">
+        <axis xyz="0 0 1" />
+        <parent link="dummy_link1"/>
+        <child link="dummy_link2"/>
+        <limit lower="-3.14" upper="3.14" effort="50" velocity="3.49" />
+      </joint> -->
+      <!-- <joint name="revolute_joint_y" type="revolute">
+        <parent link="dummy_link1"/>
+        <child link="camera_link"/>
+        <axis xyz="0 1 0"/>
+        <limit lower="-3.14" upper="3.14" effort="50" velocity="3.49" />
+      </joint>
+      <gazebo reference="dummy_link1">
+        <mu1>0.2</mu1>
+        <mu2>0.2</mu2>
+        <selfCollide>1</selfCollide>
+      </gazebo>
+      <gazebo reference="dummy_link2">
+        <mu1>0.2</mu1>
+        <mu2>0.2</mu2>
+        <selfCollide>1</selfCollide>
+      </gazebo>
+      <gazebo reference="camera_link">
+        <mu1>0.2</mu1>
+        <mu2>0.2</mu2>
+        <selfCollide>1</selfCollide>
+      </gazebo> -->
 </robot>

File: universal_robot/ur_e_description/urdf/ur.transmission.xacro (robot description, xacro)
@@ -56,5 +56,5 @@
       </actuator>
     </transmission>
-    <transmission name="${prefix}camera_link_trans">
+    <!-- <transmission name="${prefix}camera_link_trans">
       <type>transmission_interface/SimpleTransmission</type>
       <joint name="${prefix}camera_joint">
@@ -64,5 +64,32 @@
         <mechanicalReduction>1</mechanicalReduction>
       </actuator>
+    </transmission> -->
+    <transmission name="${prefix}camera_link_prismatic_z_trans">
+      <type>transmission_interface/SimpleTransmission</type>
+      <joint name="${prefix}prismatic_joint_Z">
+        <hardwareInterface>hardware_interface/EffortJointInterface</hardwareInterface>
+      </joint>
+      <actuator name="${prefix}camera_link_prismatic_z_motor">
+        <mechanicalReduction>1</mechanicalReduction>
+      </actuator>
     </transmission>
+    <transmission name="${prefix}camera_link_revolute_z_trans">
+      <type>transmission_interface/SimpleTransmission</type>
+      <joint name="${prefix}revolute_joint_z">
+        <hardwareInterface>hardware_interface/EffortJointInterface</hardwareInterface>
+      </joint>
+      <actuator name="${prefix}camera_link_revolute_z_motor">
+        <mechanicalReduction>1</mechanicalReduction>
+      </actuator>
+    </transmission>
+    <!-- <transmission name="${prefix}camera_link_revolute_y_trans">
+      <type>transmission_interface/SimpleTransmission</type>
+      <joint name="${prefix}revolute_joint_y">
+        <hardwareInterface>hardware_interface/EffortJointInterface</hardwareInterface>
+      </joint>
+      <actuator name="${prefix}camera_link_revolute_y_motor">
+        <mechanicalReduction>1</mechanicalReduction>
+      </actuator>
+    </transmission> -->
   </xacro:macro>
 </robot>

Commit message: old_camera_fixed_no_prismatic_3d_camera_introduced

File: universal_robot/ur_e_description/urdf/ur.camera.xacro (robot description, xacro)
@@ -4,89 +4,120 @@
       <color rgba="0.8 0.0 0.0 1.0"/>
     </material>
-    <xacro:property name="cameraSize" value="0.07" /> <!-- Size of square 'camera' box -->
+    <xacro:property name="cameraSize" value="0.03" /> <!-- Size of square 'camera' box -->
     <xacro:property name="cameraMass" value="0.1" /> <!-- Mass of square 'camera' box -->
-    <joint name="prismatic_joint_Z" type="prismatic">
-        <axis xyz="0 0 1" limit="-3.14 3.14" />
-        <origin xyz="0 0 1" rpy="0 0 0"/>
-        <parent link="base_link"/>
-        <child link="dummy_link1"/>
-        <limit effort="330.0" velocity="3.14"/>
-      </joint>
-      <link name="dummy_link1"/>
-      <joint name="base_link_to dummy_link1" type="fixed">
-        <parent link="base_link" />
-        <child link="dummy_link1" />
-      </joint>
-      <joint name="revolute_joint_z" type="revolute">
-        <axis xyz="0 0 1" limit="-3.14 3.14" />
-        <origin xyz="0 0 1" rpy="0 0 0"/>
-        <parent link="dummy_link1"/>
-        <child link="camera_link"/>
-        <limit effort="330.0" velocity="3.14"/>
-      </joint>
-      <link name="camera_link">
-        <collision>
-          <origin xyz="0 0 0" rpy="0 0 0"/>
+    <joint name="prismatic_joint_z" type="fixed">
+      <!-- <axis xyz="0 0 1" /> -->
+      <origin xyz="0 0 1" rpy="0 0 0"/>
+      <parent link="base_link"/>
+      <child link="camera_base"/>
+      <!-- <limit lower="-3.14" upper="3.14" effort="50" velocity="3.49" /> -->
+    </joint>
+    <link name="camera_base">
+      <inertial>
+          <origin xyz="-1.042E-08 -0.0034422 0.026198" rpy="0 0 0" />
+          <mass value="0.090334" />
+          <inertia ixx="6.8467E-05" ixy="5.9979E-12" ixz="1.3439E-12" iyy="6.5123E-05" iyz="-1.8873E-07" izz="0.00010174" />
+      </inertial>
+      <visual>
+          <origin xyz="0 0 0" rpy="0 0 0" />
           <geometry>
+              <mesh filename="package://camera_mechanism_movment/meshes/base_link.STL" />
+          </geometry>
+          <material name="">
+              <color rgba="0.79216 0.81961 0.93333 1" />
+          </material>
+      </visual>
+      <collision>
+          <origin xyz="0 0 0" rpy="0 0 0" />
+          <geometry>
+              <mesh filename="package://camera_mechanism_movment/meshes/base_link.STL" />
+          </geometry>
+      </collision>
+  </link>
+  <link name="link_1">
+      <inertial>
+          <origin xyz="-0.00274428257190968 -0.00020748847805208 0.0169598693710931" rpy="0 0 0" />
+          <mass value="0.0762928038541526" />
+          <inertia ixx="2.78524913265596E-05" ixy="1.44751279636948E-08" ixz="7.79881822675902E-07" iyy="1.38848895102569E-05" iyz="1.4640337530444E-08" izz="3.46925557643959E-05" />
+      </inertial>
+      <visual>
+          <origin xyz="0 0 0" rpy="0 0 0" />
+          <geometry>
+              <mesh filename="package://camera_mechanism_movment/meshes/link_1.STL" />
+          </geometry>
+          <material name="">
+              <color rgba="0.752941176470588 0.752941176470588 0.752941176470588 1" />
+          </material>
+      </visual>
+      <collision>
+          <origin xyz="0 0 0" rpy="0 0 0" />
+          <geometry>
+              <mesh filename="package://camera_mechanism_movment/meshes/link_1.STL" />
+          </geometry>
+      </collision>
+  </link>
+  <joint name="joint_1" type="revolute">
+      <origin xyz="0 0 0.045256" rpy="0 0 0" />
+      <parent link="camera_base" />
+      <child link="link_1" />
+      <axis xyz="0 0 -1" />
+      <limit lower="-1.5708" upper="1.5708" effort="15" velocity="137" />
+  </joint>
+  <link name="link_2">
+      <inertial>
+          <origin xyz="0.00319069336561053 0.0467174118427644 0.0302711238523648" rpy="0 0 0" />
+          <mass value="0.0760046548351893" />
+          <inertia ixx="8.75759430262867E-05" ixy="-3.75975452138231E-08" ixz="-8.26121264442182E-07" iyy="8.43979936608012E-05" iyz="3.14738619919505E-08" izz="1.01097278745386E-05" />
+      </inertial>
+      <visual>
+          <origin xyz="0 0 0" rpy="0 0 0" />
+          <geometry>
+              <mesh filename="package://camera_mechanism_movment/meshes/link_2.STL" />
+          </geometry>
+          <material name="">
+              <color rgba="0.792156862745098 0.819607843137255 0.933333333333333 1" />
+          </material>
+      </visual>
+      <collision>
+          <origin xyz="0 0 0" rpy="0 0 0" />
+          <geometry>
+              <mesh filename="package://camera_mechanism_movment/meshes/link_2.STL" />
+          </geometry>
+      </collision>
+  </link>
+  <joint name="joint_2" type="revolute">
+      <origin xyz="0.029615 -0.010178 0.021744" rpy="1.5708 0 -1.5708" />
+      <parent link="link_1" />
+      <child link="link_2" />
+      <axis xyz="0 0 1" />
+      <limit lower="-1.5708" upper="1.5708" effort="15" velocity="137" />
+  </joint>
+  <!--///////////////////////////////////////actual simulated camera/////////////////////////////-->
+  <link name="camera_link">
+    <collision>
+      <origin xyz="0 0 0" rpy="0 0 0"/>
+      <geometry>
         <box size="${cameraSize} ${cameraSize} ${cameraSize}"/>
-          </geometry>
-        </collision>
-        <visual>
-          <origin xyz="0 0 0" rpy="0 0 0"/>
-          <geometry>
+      </geometry>
+    </collision>
+    <!-- <visual>
+      <origin xyz="0 0 0" rpy="0 0 0"/>
+      <geometry>
         <box size="${cameraSize} ${cameraSize} ${cameraSize}"/>
-          </geometry>
-          <material name="red"/>
-        </visual>
-        <inertial>
-          <mass value="${cameraMass}" />
-          <origin xyz="0 0 0" rpy="0 0 0"/>
-          <box_inertia m="${cameraMass}" x="${cameraSize}" y="${cameraSize}" z="${cameraSize}"/>>
-          <inertia ixx="1e-6" ixy="0" ixz="0" iyy="1e-6" iyz="0" izz="1e-6" />
-        </inertial>
-      </link>
-      <!-- <link name="dummy_link1"/>
-      <link name="dummy_link2"/>
-      <joint name="base_link_to dummy_link1" type="fixed">
-        <parent link="base_link" />
-        <child link="dummy_link1" />
-      </joint> -->
-      <!-- <joint name="base_link_to dummy_link2" type="fixed">
-        <parent link="world" />
-        <child link="dummy_link2" />
-      </joint>   -->
-      <!-- <joint name="prismatic_joint_Z" type="prismatic">
-        <parent link="base_link"/>
-        <child link="dummy_link1"/>
-        <origin xyz="0 0 1" rpy="0 0 0"/>
-        <axis xyz="0 0 1"/>
-        <limit lower="-2" upper="2" effort="50" velocity="3.49" />
-      </joint>
-      <joint name="revolute_joint_z" type="revolute">
-        <axis xyz="0 0 1" />
-        <parent link="dummy_link1"/>
-        <child link="dummy_link2"/>
-        <limit lower="-3.14" upper="3.14" effort="50" velocity="3.49" />
-      </joint> -->
-      <!-- <joint name="revolute_joint_y" type="revolute">
-        <parent link="dummy_link1"/>
-        <child link="camera_link"/>
-        <axis xyz="0 1 0"/>
-        <limit lower="-3.14" upper="3.14" effort="50" velocity="3.49" />
-      </joint>
-      <gazebo reference="dummy_link1">
-        <mu1>0.2</mu1>
-        <mu2>0.2</mu2>
-        <selfCollide>1</selfCollide>
-      </gazebo>
-      <gazebo reference="dummy_link2">
-        <mu1>0.2</mu1>
-        <mu2>0.2</mu2>
-        <selfCollide>1</selfCollide>
-      </gazebo>
-      <gazebo reference="camera_link">
-        <mu1>0.2</mu1>
-        <mu2>0.2</mu2>
-        <selfCollide>1</selfCollide>
-      </gazebo> -->
+      </geometry>
+      <material name="red"/>
+    </visual> -->
+    <inertial>
+      <mass value="${cameraMass}" />
+      <origin xyz="0 0 0" rpy="0 0 0"/>
+      <box_inertia m="${cameraMass}" x="${cameraSize}" y="${cameraSize}" z="${cameraSize}" />
+      <inertia ixx="1e-6" ixy="0" ixz="0" iyy="1e-6" iyz="0" izz="1e-6" />
+    </inertial>
+  </link>
+  <joint name="camera_joint" type="fixed">
+    <axis xyz="0 1 0" />
+    <origin xyz=".02 .05 .0342" rpy="-1.5708 0 0"/>
+    <parent link="link_2"/>
+    <child link="camera_link"/>
+  </joint>
 </robot>

File: universal_robot/ur_e_description/urdf/ur.transmission.xacro (robot description, xacro)
@@ -65,14 +65,15 @@
       </actuator>
     </transmission> -->
-    <transmission name="${prefix}camera_link_prismatic_z_trans">
+    <!-- <transmission name="${prefix}camera_link_prismatic_z_trans">
       <type>transmission_interface/SimpleTransmission</type>
-      <joint name="${prefix}prismatic_joint_Z">
+      <joint name="${prefix}prismatic_joint_z">
         <hardwareInterface>hardware_interface/EffortJointInterface</hardwareInterface>
       </joint>
       <actuator name="${prefix}camera_link_prismatic_z_motor">
+        <hardwareInterface>hardware_interface/EffortJointInterface</hardwareInterface>
         <mechanicalReduction>1</mechanicalReduction>
       </actuator>
-    </transmission>
-    <transmission name="${prefix}camera_link_revolute_z_trans">
+    </transmission> -->
+    <!-- <transmission name="${prefix}camera_link_revolute_z_trans">
       <type>transmission_interface/SimpleTransmission</type>
       <joint name="${prefix}revolute_joint_z">
@@ -80,8 +81,9 @@
       </joint>
       <actuator name="${prefix}camera_link_revolute_z_motor">
+        <hardwareInterface>hardware_interface/EffortJointInterface</hardwareInterface>
         <mechanicalReduction>1</mechanicalReduction>
       </actuator>
     </transmission>
-    <!-- <transmission name="${prefix}camera_link_revolute_y_trans">
+    <transmission name="${prefix}camera_link_revolute_y_trans">
       <type>transmission_interface/SimpleTransmission</type>
       <joint name="${prefix}revolute_joint_y">
@@ -89,7 +91,28 @@
       </joint>
       <actuator name="${prefix}camera_link_revolute_y_motor">
+        <hardwareInterface>hardware_interface/EffortJointInterface</hardwareInterface>
         <mechanicalReduction>1</mechanicalReduction>
       </actuator>
     </transmission> -->
+    <transmission name="trans_joint_1">
+      <type>transmission_interface/SimpleTransmission</type>
+      <joint name="joint_1">
+          <hardwareInterface>hardware_interface/EffortJointInterface</hardwareInterface>
+      </joint>
+      <actuator name="joint_1_motor">
+          <hardwareInterface>hardware_interface/EffortJointInterface</hardwareInterface>
+          <mechanicalReduction>1</mechanicalReduction>
+      </actuator>
+  </transmission>
+  <transmission name="trans_joint_2">
+      <type>transmission_interface/SimpleTransmission</type>
+      <joint name="joint_2">
+          <hardwareInterface>hardware_interface/EffortJointInterface</hardwareInterface>
+      </joint>
+      <actuator name="joint_2_motor">
+          <hardwareInterface>hardware_interface/EffortJointInterface</hardwareInterface>
+          <mechanicalReduction>1</mechanicalReduction>
+      </actuator>
+  </transmission>
   </xacro:macro>
 </robot>

File: universal_robot/ur_e_description/urdf/ur10e.urdf.xacro (robot description, xacro)
@@ -9,4 +9,6 @@
   <xacro:include filename="$(find ur_e_description)/urdf/ur.camera.gazebo"/>
   <xacro:include filename="$(find ur_e_description)/urdf/ur.camera.xacro"/>
+  <xacro:include filename="$(find ur_e_description)/urdf/ur.3dcamera.gazebo"/>
+  <xacro:include filename="$(find ur_e_description)/urdf/ur.3dcamera.xacro"/>
   <xacro:macro name="cylinder_inertial" params="radius length mass *origin">
     <inertial>
@@ -320,4 +322,5 @@
     <xacro:ur_arm_transmission prefix="${prefix}" />
     <xacro:ur_arm_gazebo prefix="${prefix}" />
+    <xacro:macro name="ur_camera" params="prefix"/>
     <!-- ROS base_link to UR 'Base' Coordinates transform -->
     <link name="${prefix}base"/>
