Commit message: 3d_camera_output_shown_in_correct_pos

File: universal_robot/ur_e_description/urdf/ur.3dcamera.xacro (robot description, xacro)
@@ -4,6 +4,8 @@
       <color rgba="0.8 0.0 0.0 1.0"/>
     </material>
-    <xacro:property name="cameraSize" value="0.03" /> <!-- Size of square 'camera' box -->
-    <xacro:property name="cameraMass" value="0.1" /> <!-- Mass of square 'camera' box -->
+    <xacro:property name="cameraSize_x" value="0.142" /> <!-- Size of square 'camera' box -->
+    <xacro:property name="cameraSize_y" value="0.26" /> <!-- Size of square 'camera' box -->
+    <xacro:property name="cameraSize_z" value="0.065" /> <!-- Size of square 'camera' box -->
+    <xacro:property name="cameraMass" value="1.9" /> <!-- Mass of square 'camera' box -->
   <!--///////////////////////////////////////simulated 3dcamera/////////////////////////////-->
   <link name="3d_camera_link">
@@ -11,5 +13,5 @@
       <origin xyz="0 0 0" rpy="0 0 0"/>
       <geometry>
-        <box size="${cameraSize} ${cameraSize} ${cameraSize}"/>
+        <box size="${cameraSize_x} ${cameraSize_y} ${cameraSize_z}"/>
       </geometry>
     </collision>
@@ -17,5 +19,5 @@
       <origin xyz="0 0 0" rpy="0 0 0"/>
       <geometry>
-        <box size="${cameraSize} ${cameraSize} ${cameraSize}"/>
+        <box size="${cameraSize_x} ${cameraSize_y} ${cameraSize_z}"/>
       </geometry>
       <material name="3d_red"/>
@@ -24,13 +26,19 @@
       <mass value="${cameraMass}" />
       <origin xyz="0 0 0" rpy="0 0 0"/>
-      <box_inertia m="${cameraMass}" x="${cameraSize}" y="${cameraSize}" z="${cameraSize}" />
+      <box_inertia m="${cameraMass}" x="${cameraSize_x}" y="${cameraSize_y}" z="${cameraSize_z}" />
       <inertia ixx="1e-6" ixy="0" ixz="0" iyy="1e-6" iyz="0" izz="1e-6" />
     </inertial>
   </link>
   <joint name="3d_camera_joint" type="fixed">
-    <axis xyz="0 1 0" />
-    <origin xyz=".2 0 0" rpy="-1.5708 0 0"/>
+    <axis xyz="1 0 0" />
+    <origin xyz="-0.1 0 0" rpy="0 -1.5708 0"/>
     <parent link="wrist_3_link"/>
     <child link="3d_camera_link"/>
   </joint>
+  <joint name="camera_optical_joint" type="fixed">
+    <origin xyz="0 0 0" rpy="-1.5708 0 -1.5708"/>
+    <parent link="3d_camera_link"/>
+    <child link="camera_frame_optical"/>
+  </joint>
+  <link name="camera_frame_optical"/>
 </robot>

Commit message: changed position of 3d camera

File: universal_robot/ur_e_description/urdf/ur.3dcamera.xacro (robot description, xacro)
@@ -32,5 +32,5 @@
   <joint name="3d_camera_joint" type="fixed">
     <axis xyz="1 0 0" />
-    <origin xyz="-0.1 0 0" rpy="0 -1.5708 0"/>
+    <origin xyz="0 0 0.15" rpy="0 0 3.14159"/>
     <parent link="wrist_3_link"/>
     <child link="3d_camera_link"/>

Commit message: orientation fix

File: universal_robot/ur_e_description/urdf/ur.3dcamera.xacro (robot description, xacro)
@@ -32,5 +32,5 @@
   <joint name="3d_camera_joint" type="fixed">
     <axis xyz="1 0 0" />
-    <origin xyz="0 0 0.15" rpy="0 0 3.14159"/>
+    <origin xyz="0 0 0.15" rpy="0 0 1.5708"/>
     <parent link="wrist_3_link"/>
     <child link="3d_camera_link"/>
