Commit message: exo_plus_hand_bringup

File: exoskelaton_model/urdf/exoskelaton_model.urdf (robot description, URDF)
Before this commit: robot exoskelaton_model, 7 links, 6 joints
Links:
- link base_link: mass 2.5151 -> 2.51510979215834; geometry collision mesh filename=package://exoskelaton_model_2/meshes/base_link.STL; visual mesh filename=package://exoskelaton_model_2/meshes/base_link.STL
- link link_1: geometry collision mesh filename=package://exoskelaton_model_2/meshes/link_1.STL; visual mesh filename=package://exoskelaton_model_2/meshes/link_1.STL
- link link_2: geometry collision mesh filename=package://exoskelaton_model_2/meshes/link_2.STL; visual mesh filename=package://exoskelaton_model_2/meshes/link_2.STL
- link link_3: geometry collision mesh filename=package://exoskelaton_model_2/meshes/link_3.STL; visual mesh filename=package://exoskelaton_model_2/meshes/link_3.STL
- link link_4: geometry collision mesh filename=package://exoskelaton_model_2/meshes/link_4.STL; visual mesh filename=package://exoskelaton_model_2/meshes/link_4.STL
- link link_5: geometry collision mesh filename=package://exoskelaton_model_2/meshes/link_5.STL; visual mesh filename=package://exoskelaton_model_2/meshes/link_5.STL
Joints:
- joint joint_1: origin xyz=-0.15577 0.0088052 -0.26586 rpy=-0.00036153 -0.00029771 -3.1416 -> xyz=-0.15576841452816 0.00880518561429395 -0.265864926099811 rpy=-0.00036152630959631 -0.000297710155103675 -3.14159254595974
- joint joint_2: origin xyz=-0.03876 0.11791 0.13076 rpy=-3.1238 -1.5708 3.126 -> xyz=-0.0385000000000007 0.117999999999999 0.130760035281312 rpy=-0.037127716917956 -1.57079631189374 0.0371631202033193
- joint joint_3: origin xyz=-0.03366 0.20656 0.046 rpy=1.5708 0 -1.6211 -> xyz=-0.0440000000000005 0.204606049200406 0.045999999999999 rpy=1.57079632679491 0 -1.5707963267949
- joint joint_4: axis 0 0 -1 -> 0.00029771017016183 0 -0.999999955684326; origin xyz=0.0027746 0.20467 0.047 rpy=1.5708 0 1.7195 -> xyz=0.0330000000000062 0.202007049200406 0.0469999999999915 rpy=1.5707963267949 0 1.57109403696946
- joint joint_5: origin xyz=-0.13159 0.24476 0.0099608 rpy=-0.00024377 0.0001709 2.1822 -> xyz=0.032755858725567 0.275947208661753 0.0100097521958599 rpy=-0.000297710174561625 0 1.57079632679491

Commit message: fixed exoskelton package meshes folder path

File: exoskelaton_model/urdf/exoskelaton_model.urdf (robot description, URDF)
Before this commit: robot exoskelaton_model, 7 links, 6 joints
Links:
- link base_link: geometry collision mesh filename=package://exoskelaton_model/meshes/base_link.STL; visual mesh filename=package://exoskelaton_model/meshes/base_link.STL
- link link_1: geometry collision mesh filename=package://exoskelaton_model/meshes/link_1.STL; visual mesh filename=package://exoskelaton_model/meshes/link_1.STL
- link link_2: geometry collision mesh filename=package://exoskelaton_model/meshes/link_2.STL; visual mesh filename=package://exoskelaton_model/meshes/link_2.STL
- link link_3: geometry collision mesh filename=package://exoskelaton_model/meshes/link_3.STL; visual mesh filename=package://exoskelaton_model/meshes/link_3.STL
- link link_4: geometry collision mesh filename=package://exoskelaton_model/meshes/link_4.STL; visual mesh filename=package://exoskelaton_model/meshes/link_4.STL
- link link_5: geometry collision mesh filename=package://exoskelaton_model/meshes/link_5.STL; visual mesh filename=package://exoskelaton_model/meshes/link_5.STL
